Commit message: add gazebo gripper plugin

File: ur_description/urdf/ur10_joint_limited_robot_2f85.urdf.xacro (robot description, xacro)
@@ -15,4 +15,7 @@
     <origin xyz="0 0 0" rpy="0 ${-pi/2.0} 0"/>
   </xacro:robotiq_85_gripper>
+  <!-- Gazebo gripper plugin -->
+  <xacro:include filename="$(find robotiq_description)/urdf/robotiq_85_gripper.gazebo.xacro" />
+  <xacro:robotiq_85_gripper_gazebo prefix=""/>
   <!-- end_effector cord-->
   <link name="tool_gripper"/>
@@ -22,57 +25,3 @@
     <origin rpy="0 0 0" xyz="0.14 0 0"/>
   </joint>
-  <!-- realsense d435 (hand-eye) -->
-  <xacro:include filename="$(find realsense2_description)/urdf/_d435.urdf.xacro" />
-  <xacro:sensor_d435 name="hand_eye" topics_ns="hand_eye" parent="ee_link" publish_pointcloud="false">
-    <origin xyz="0 0 0.1" rpy="0 0.35 0" />
-  </xacro:sensor_d435>
-  <!-- realsense d435 (side_camera) -->
-  <xacro:include filename="$(find realsense2_description)/urdf/_d435.urdf.xacro" />
-  <xacro:sensor_d435 name="side_camera" topics_ns="side_camera" parent="base_link" publish_pointcloud="false">
-    <origin xyz="1 0.6 0.3" rpy="0 0 ${pi}" />
-  </xacro:sensor_d435>
-  <!-- realsense d435 (front_camera) -->
-  <xacro:include filename="$(find realsense2_description)/urdf/_d435.urdf.xacro" />
-  <xacro:sensor_d435 name="front_camera" topics_ns="front_camera" parent="base_link" publish_pointcloud="false">
-    <origin xyz="0.2 1.25 0.3" rpy="0 0 ${-pi/2.0}" />
-  </xacro:sensor_d435>
-  <!-- Gazebo grasping plugin
-      grasp_plugin False = gazebo_gripper
-      grasp_plugin True = custom gazebo_grasp_fix
-  -->
-  <xacro:arg name="grasp_plugin" default="true" />
-  <xacro:if value="$(arg grasp_plugin)">
-    <gazebo>
-      <plugin name="gazebo_grasp_fix" filename="libgazebo_grasp_fix.so">
-            <arm>
-              <arm_name>robotiq_85</arm_name>
-              <palm_link>tool0</palm_link>
-              <gripper_link>robotiq_85_left_finger_tip_link</gripper_link>
-              <gripper_link>robotiq_85_right_finger_tip_link</gripper_link>
-            </arm>
-          <forces_angle_tolerance>100</forces_angle_tolerance>
-          <update_rate>100</update_rate>
-          <grip_count_threshold>5</grip_count_threshold>
-          <max_grip_count>30</max_grip_count>
-          <release_tolerance>0.0015</release_tolerance>
-          <disable_collisions_on_attach>false</disable_collisions_on_attach>
-          <contact_topic>__default_topic__</contact_topic>
-        </plugin>
-    </gazebo>
-  </xacro:if>
-  <xacro:unless value="$(arg grasp_plugin)">
-    <gazebo>
-      <gripper name="gazebo_gripper">
-        <grasp_check>
-          <attach_steps>2</attach_steps>
-          <detach_steps>2</detach_steps>
-          <min_contact_count>3</min_contact_count>
-        </grasp_check>
-        <gripper_link>robotiq_85_left_finger_tip_link</gripper_link>
-        <gripper_link>robotiq_85_right_finger_tip_link</gripper_link>
-        <palm_link>robotiq_85_base_link</palm_link>
-      </gripper>
-    </gazebo>
-  </xacro:unless>
-  <!-- Gazebo grasping plugin -->
 </robot>

File: ur_description/urdf/ur10_robot_2f85.urdf.xacro (robot description, xacro)
@@ -15,4 +15,7 @@
     <origin xyz="0 0 0" rpy="0 ${-pi/2.0} 0"/>
   </xacro:robotiq_85_gripper>
+  <!-- Gazebo gripper plugin -->
+  <xacro:include filename="$(find robotiq_description)/urdf/robotiq_85_gripper.gazebo.xacro" />
+  <xacro:robotiq_85_gripper_gazebo prefix=""/>
   <!-- end_effector cord-->
   <link name="tool_gripper"/>
@@ -22,8 +25,3 @@
     <origin rpy="0 0 0" xyz="0.14 0 0"/>
   </joint>
-  <!-- realsense d435 -->
-  <xacro:include filename="$(find realsense2_description)/urdf/_d435.urdf.xacro" />
-  <xacro:sensor_d435 name="camera" topics_ns="camera" parent="ee_link" publish_pointcloud="false">
-    <origin xyz="0 0 0.1" rpy="0 0.35 0" />
-  </xacro:sensor_d435>
 </robot>
